Commit message: Add Walk and Kick env for T1 and K1
- Also update stand-up env with latest changes
- Also add T1 and K1 walk and kick policies + c++ code reference

File: IsaacGymRL/resources/K1/Ball_K1_locomotion_feet_box_left_bias.urdf (robot description, URDF)
Before this commit: robot K1, 23 links, 22 joints
Links:
- link Head_1: geometry visual mesh filename=meshes/Head_1.STL
- link Head_2: geometry visual mesh filename=meshes/Head_2.STL
- link Left_Arm_2: geometry visual mesh filename=meshes/Left_Arm_2.STL
- link Left_Arm_3: geometry visual mesh filename=meshes/Left_Arm_3.STL
- link Left_Shank: geometry collision box size=0.08 0.07 0.13; collision cylinder length=0.07 radius=0.045
- link Right_Arm_2: geometry visual mesh filename=meshes/Right_Arm_2.STL
- link Right_Arm_3: geometry visual mesh filename=meshes/Right_Arm_3.STL
- link Right_Shank: geometry collision box size=0.08 0.07 0.13; collision cylinder length=0.07 radius=0.045
- link left_foot_link: geometry collision box size=0.01 0.005 0.01; collision box size=0.180 0.07 0.016
- link left_hand_link: geometry visual mesh filename=meshes/Left_Arm_4.STL
- link right_foot_link: geometry collision box size=0.01 0.005 0.01; collision box size=0.180 0.07 0.016
- link right_hand_link: geometry visual mesh filename=meshes/Right_Arm_4.STL
Joints:
- joint AAHead_yaw: type revolute -> fixed
- joint ALeft_Shoulder_Pitch: type revolute -> fixed
- joint ARight_Shoulder_Pitch: type revolute -> fixed
- joint Head_pitch: type revolute -> fixed
- joint Left_Elbow_Pitch: type revolute -> fixed
- joint Left_Elbow_Yaw: type revolute -> fixed
- joint Left_Shoulder_Roll: origin xyz=0.0025 0.068 -0.0135 rpy=0 0 0 -> xyz=0.0025 0.068 -0.0135 rpy=-1.35 0 0; type revolute -> fixed
- joint Right_Elbow_Pitch: type revolute -> fixed
- joint Right_Elbow_Yaw: type revolute -> fixed
- joint Right_Shoulder_Roll: origin xyz=0.0025 -0.068 -0.0135 rpy=0 0 0 -> xyz=0.0025 -0.068 -0.0135 rpy=1.35 0 0; type revolute -> fixed

File: IsaacGymRL/resources/K1/Ball_K1_locomotion_feet_box_right_bias.urdf (robot description, URDF)
Before this commit: robot K1, 23 links, 22 joints
Links:
- link Head_1: geometry visual mesh filename=meshes/Head_1.STL
- link Head_2: geometry visual mesh filename=meshes/Head_2.STL
- link Left_Arm_2: geometry visual mesh filename=meshes/Left_Arm_2.STL
- link Left_Arm_3: geometry visual mesh filename=meshes/Left_Arm_3.STL
- link Left_Shank: geometry collision box size=0.08 0.07 0.13; collision cylinder length=0.07 radius=0.045
- link Right_Arm_2: geometry visual mesh filename=meshes/Right_Arm_2.STL
- link Right_Arm_3: geometry visual mesh filename=meshes/Right_Arm_3.STL
- link Right_Shank: geometry collision box size=0.08 0.07 0.13; collision cylinder length=0.07 radius=0.045
- link left_foot_link: geometry collision box size=0.01 0.005 0.01; collision box size=0.180 0.07 0.016
- link left_hand_link: geometry visual mesh filename=meshes/Left_Arm_4.STL
- link right_foot_link: geometry collision box size=0.01 0.005 0.01; collision box size=0.180 0.07 0.016
- link right_hand_link: geometry visual mesh filename=meshes/Right_Arm_4.STL
Joints:
- joint AAHead_yaw: type revolute -> fixed
- joint ALeft_Shoulder_Pitch: type revolute -> fixed
- joint ARight_Shoulder_Pitch: type revolute -> fixed
- joint Head_pitch: type revolute -> fixed
- joint Left_Elbow_Pitch: type revolute -> fixed
- joint Left_Elbow_Yaw: type revolute -> fixed
- joint Left_Shoulder_Roll: origin xyz=0.0025 0.068 -0.0135 rpy=0 0 0 -> xyz=0.0025 0.068 -0.0135 rpy=-1.35 0 0; type revolute -> fixed
- joint Right_Elbow_Pitch: type revolute -> fixed
- joint Right_Elbow_Yaw: type revolute -> fixed
- joint Right_Shoulder_Roll: origin xyz=0.0025 -0.068 -0.0135 rpy=0 0 0 -> xyz=0.0025 -0.068 -0.0135 rpy=1.35 0 0; type revolute -> fixed

File: IsaacGymRL/resources/K1/K1_arms_locomotion.urdf (robot description, URDF)
Before this commit: robot K1, 23 links, 22 joints
Links:
- link Head_1: geometry visual mesh filename=meshes/Head_1.STL
- link Head_2: geometry visual mesh filename=meshes/Head_2.STL
- link Left_Arm_2: geometry visual mesh filename=meshes/Left_Arm_2.STL
- link Right_Arm_2: geometry visual mesh filename=meshes/Right_Arm_2.STL
Joints:
- joint AAHead_yaw: type revolute -> fixed
- joint Head_pitch: type revolute -> fixed

File: IsaacGymRL/resources/K1/K1_arms_locomotion_feet_box.urdf (robot description, URDF)
Before this commit: robot K1, 23 links, 22 joints
Links:
- link Head_1: geometry visual mesh filename=meshes/Head_1.STL
- link Head_2: geometry visual mesh filename=meshes/Head_2.STL
- link Left_Shank: geometry collision box size=0.06 0.06 0.10; collision cylinder length=0.07 radius=0.045
- link Right_Shank: geometry collision box size=0.06 0.06 0.1; collision cylinder length=0.07 radius=0.045
- link left_foot_link: geometry collision box size=0.180 0.07 0.032; visual mesh filename=meshes/Left_Foot.STL
- link right_foot_link: geometry collision box size=0.180 0.07 0.032; visual mesh filename=meshes/Right_Foot.STL
Joints:
- joint AAHead_yaw: type revolute -> fixed
- joint Head_pitch: type revolute -> fixed

File: IsaacGymRL/resources/K1/K1_locomotion.urdf (robot description, URDF)
Before this commit: robot K1, 23 links, 22 joints
Links:
- link Head_1: geometry visual mesh filename=meshes/Head_1.STL
- link Head_2: geometry visual mesh filename=meshes/Head_2.STL
- link Left_Arm_2: geometry visual mesh filename=meshes/Left_Arm_2.STL
- link Left_Arm_3: geometry visual mesh filename=meshes/Left_Arm_3.STL
- link Left_Shank: geometry collision box size=0.0001 0.0001 0.0001; collision mesh filename=meshes/Left_Shank.STL scale=1 1 0.8
- link Right_Arm_2: geometry visual mesh filename=meshes/Right_Arm_2.STL
- link Right_Arm_3: geometry visual mesh filename=meshes/Right_Arm_3.STL
- link Right_Shank: geometry collision box size=0.0001 0.0001 0.0001; collision mesh filename=meshes/Right_Shank.STL scale=1 1 0.8
- link left_hand_link: geometry visual mesh filename=meshes/Left_Arm_4.STL
- link right_hand_link: geometry visual mesh filename=meshes/Right_Arm_4.STL
Joints:
- joint AAHead_yaw: type revolute -> fixed
- joint ALeft_Shoulder_Pitch: type revolute -> fixed
- joint ARight_Shoulder_Pitch: type revolute -> fixed
- joint Head_pitch: type revolute -> fixed
- joint Left_Elbow_Pitch: type revolute -> fixed
- joint Left_Elbow_Yaw: type revolute -> fixed
- joint Left_Shoulder_Roll: origin xyz=0.0025 0.068 -0.0135 rpy=0 0 0 -> xyz=0.0025 0.068 -0.0135 rpy=-1.35 0 0; type revolute -> fixed
- joint Right_Elbow_Pitch: type revolute -> fixed
- joint Right_Elbow_Yaw: type revolute -> fixed
- joint Right_Shoulder_Roll: origin xyz=0.0025 -0.068 -0.0135 rpy=0 0 0 -> xyz=0.0025 -0.068 -0.0135 rpy=1.35 0 0; type revolute -> fixed

File: IsaacGymRL/resources/K1/K1_locomotion_all_joints_simple_2.urdf (robot description, URDF)
Before this commit: robot K1, 23 links, 22 joints
Links:
- link Head_2: geometry collision mesh filename=meshes/Head_2.STL scale=1 1 0.8; visual mesh filename=meshes/Head_2.STL
- link Left_Arm_1: geometry collision cylinder length=0.00001 radius=0.00001; visual mesh filename=meshes/Left_Arm_1.STL
- link Left_Hip_Pitch: geometry collision cylinder length=0.00001 radius=0.00001; visual mesh filename=meshes/Left_Hip_Pitch.STL
- link Left_Hip_Roll: geometry collision cylinder length=0.05 radius=0.02; visual mesh filename=meshes/Left_Hip_Roll.STL
- link Right_Arm_1: geometry collision cylinder length=0.0001 radius=0.00001; visual mesh filename=meshes/Right_Arm_1.STL
- link Right_Hip_Pitch: geometry collision cylinder length=0.00001 radius=0.00001; visual mesh filename=meshes/Right_Hip_Pitch.STL
- link Right_Hip_Roll: geometry collision cylinder length=0.05 radius=0.02; visual mesh filename=meshes/Right_Hip_Roll.STL
- link Trunk: geometry collision cylinder length=0.1 radius=0.05; collision mesh filename=meshes/Trunk.STL scale=1.0 1.0 1.0
- link left_foot_link: geometry collision box size=0.180 0.07 0.032; visual mesh filename=meshes/Left_Foot.STL
- link right_foot_link: geometry collision box size=0.180 0.07 0.032; visual mesh filename=meshes/Right_Foot.STL

File: IsaacGymRL/resources/K1/K1_locomotion_feet_box.urdf (robot description, URDF)
Before this commit: robot K1, 23 links, 22 joints
Links:
- link Head_1: geometry visual mesh filename=meshes/Head_1.STL
- link Head_2: geometry visual mesh filename=meshes/Head_2.STL
- link Left_Arm_2: geometry visual mesh filename=meshes/Left_Arm_2.STL
- link Left_Arm_3: geometry visual mesh filename=meshes/Left_Arm_3.STL
- link Left_Shank: geometry collision box size=0.01 0.08 0.05; collision box size=0.1 0.08 0.12
- link Right_Arm_2: geometry visual mesh filename=meshes/Right_Arm_2.STL
- link Right_Arm_3: geometry visual mesh filename=meshes/Right_Arm_3.STL
- link Right_Shank: geometry collision box size=0.01 0.08 0.05; collision box size=0.1 0.08 0.12
- link left_foot_link: geometry collision box size=0.180 0.07 0.016; visual mesh filename=meshes/Left_Foot.STL
- link left_hand_link: geometry visual mesh filename=meshes/Left_Arm_4.STL
- link right_foot_link: geometry collision box size=0.180 0.07 0.016; visual mesh filename=meshes/Right_Foot.STL
- link right_hand_link: geometry visual mesh filename=meshes/Right_Arm_4.STL
Joints:
- joint AAHead_yaw: type revolute -> fixed
- joint ALeft_Shoulder_Pitch: type revolute -> fixed
- joint ARight_Shoulder_Pitch: type revolute -> fixed
- joint Head_pitch: type revolute -> fixed
- joint Left_Elbow_Pitch: type revolute -> fixed
- joint Left_Elbow_Yaw: type revolute -> fixed
- joint Left_Shoulder_Roll: origin xyz=0.0025 0.068 -0.0135 rpy=0 0 0 -> xyz=0.0025 0.068 -0.0135 rpy=-1.35 0 0; type revolute -> fixed
- joint Right_Elbow_Pitch: type revolute -> fixed
- joint Right_Elbow_Yaw: type revolute -> fixed
- joint Right_Shoulder_Roll: origin xyz=0.0025 -0.068 -0.0135 rpy=0 0 0 -> xyz=0.0025 -0.068 -0.0135 rpy=1.35 0 0; type revolute -> fixed

File: IsaacGymRL/resources/T1/Ball_T1_locomotion_feet_box_left_bias.urdf (robot description, URDF)
Before this commit: robot T1, 24 links, 23 joints
Links:
- link AL1: geometry visual mesh filename=meshes/AL1.STL
- link AL2: geometry visual mesh filename=meshes/AL2.STL
- link AL3: geometry visual mesh filename=meshes/AL3.STL
- link AR1: geometry visual mesh filename=meshes/AR1.STL
- link AR2: geometry visual mesh filename=meshes/AR2.STL
- link AR3: geometry visual mesh filename=meshes/AR3.STL
- link Ankle_Cross_Left: geometry visual mesh filename=meshes/Ankle_Cross_Left.STL
- link Ankle_Cross_Right: geometry visual mesh filename=meshes/Ankle_Cross_Right.STL
- link H1: geometry visual mesh filename=meshes/H1.STL
- link H2: geometry visual mesh filename=meshes/H2.STL
- link Hip_Pitch_Left: geometry visual mesh filename=meshes/Hip_Pitch_Left.STL
- link Hip_Pitch_Right: geometry visual mesh filename=meshes/Hip_Pitch_Right.STL
- link Hip_Roll_Left: geometry visual mesh filename=meshes/Hip_Roll_Left.STL
- link Hip_Roll_Right: geometry visual mesh filename=meshes/Hip_Roll_Right.STL
- link Hip_Yaw_Left: geometry collision cylinder length=0.16 radius=0.05; visual mesh filename=meshes/Hip_Yaw_Left.STL
- link Hip_Yaw_Right: geometry collision cylinder length=0.16 radius=0.05; visual mesh filename=meshes/Hip_Yaw_Right.STL
- link Shank_Left: geometry collision cylinder length=0.18 radius=0.06; visual mesh filename=meshes/Shank_Left.STL
- link Shank_Right: geometry collision cylinder length=0.18 radius=0.06; visual mesh filename=meshes/Shank_Right.STL
- link Trunk: geometry collision box size=0.15 0.2 0.3; visual mesh filename=meshes/Trunk.STL
- link Waist: geometry visual mesh filename=meshes/Waist.STL
- link left_foot_link: geometry collision box size=0.01 0.005 0.01; collision box size=0.223 0.1 0.03
- link left_hand_link: geometry visual mesh filename=meshes/left_hand_link.STL
- link right_foot_link: geometry collision box size=0.01 0.005 0.01; collision box size=0.223 0.1 0.03
- link right_hand_link: geometry visual mesh filename=meshes/right_hand_link.STL
Joints:
- joint AAHead_yaw: type revolute -> fixed
- joint Head_pitch: type revolute -> fixed
- joint Left_Elbow_Pitch: type revolute -> fixed
- joint Left_Elbow_Yaw: origin xyz=0 0.1471 0 rpy=0 0 0 -> xyz=0 0.1471 0 rpy=0 0 -0.5; type revolute -> fixed
- joint Left_Shoulder_Pitch: origin xyz=0.0575 0.1063 0.219 rpy=0 0 0 -> xyz=0.0575 0.1063 0.219 rpy=0 0.2 0; type revolute -> fixed
- joint Left_Shoulder_Roll: origin xyz=0 0.047 0 rpy=0.0 0 0 -> xyz=0 0.047 0 rpy=-1.35 0 0; type revolute -> fixed
- joint Right_Elbow_Pitch: type revolute -> fixed
- joint Right_Elbow_Yaw: origin xyz=0 -0.1471 0 rpy=0 0 0 -> xyz=0 -0.1471 0 rpy=0 0 0.5; type revolute -> fixed
- joint Right_Shoulder_Pitch: origin xyz=0.0575 -0.1063 0.219 rpy=0 0 0 -> xyz=0.0575 -0.1063 0.219 rpy=0 0.2 0; type revolute -> fixed
- joint Right_Shoulder_Roll: origin xyz=0 -0.047 0 rpy=0 0 0 -> xyz=0 -0.047 0 rpy=1.35 0 0; type revolute -> fixed

File: IsaacGymRL/resources/T1/Ball_T1_locomotion_feet_box_right_bias.urdf (robot description, URDF)
Before this commit: robot T1, 24 links, 23 joints
Links:
- link AL1: geometry visual mesh filename=meshes/AL1.STL
- link AL2: geometry visual mesh filename=meshes/AL2.STL
- link AL3: geometry visual mesh filename=meshes/AL3.STL
- link AR1: geometry visual mesh filename=meshes/AR1.STL
- link AR2: geometry visual mesh filename=meshes/AR2.STL
- link AR3: geometry visual mesh filename=meshes/AR3.STL
- link Ankle_Cross_Left: geometry visual mesh filename=meshes/Ankle_Cross_Left.STL
- link Ankle_Cross_Right: geometry visual mesh filename=meshes/Ankle_Cross_Right.STL
- link H1: geometry visual mesh filename=meshes/H1.STL
- link H2: geometry visual mesh filename=meshes/H2.STL
- link Hip_Pitch_Left: geometry visual mesh filename=meshes/Hip_Pitch_Left.STL
- link Hip_Pitch_Right: geometry visual mesh filename=meshes/Hip_Pitch_Right.STL
- link Hip_Roll_Left: geometry visual mesh filename=meshes/Hip_Roll_Left.STL
- link Hip_Roll_Right: geometry visual mesh filename=meshes/Hip_Roll_Right.STL
- link Hip_Yaw_Left: geometry collision cylinder length=0.16 radius=0.05; visual mesh filename=meshes/Hip_Yaw_Left.STL
- link Hip_Yaw_Right: geometry collision cylinder length=0.16 radius=0.05; visual mesh filename=meshes/Hip_Yaw_Right.STL
- link Shank_Left: geometry collision cylinder length=0.18 radius=0.06; visual mesh filename=meshes/Shank_Left.STL
- link Shank_Right: geometry collision cylinder length=0.18 radius=0.06; visual mesh filename=meshes/Shank_Right.STL
- link Trunk: geometry collision box size=0.15 0.2 0.3; visual mesh filename=meshes/Trunk.STL
- link Waist: geometry visual mesh filename=meshes/Waist.STL
- link left_foot_link: geometry collision box size=0.01 0.005 0.01; collision box size=0.223 0.1 0.03
- link left_hand_link: geometry visual mesh filename=meshes/left_hand_link.STL
- link right_foot_link: geometry collision box size=0.01 0.005 0.01; collision box size=0.223 0.1 0.03
- link right_hand_link: geometry visual mesh filename=meshes/right_hand_link.STL
Joints:
- joint AAHead_yaw: type revolute -> fixed
- joint Head_pitch: type revolute -> fixed
- joint Left_Elbow_Pitch: type revolute -> fixed
- joint Left_Elbow_Yaw: origin xyz=0 0.1471 0 rpy=0 0 0 -> xyz=0 0.1471 0 rpy=0 0 -0.5; type revolute -> fixed
- joint Left_Shoulder_Pitch: origin xyz=0.0575 0.1063 0.219 rpy=0 0 0 -> xyz=0.0575 0.1063 0.219 rpy=0 0.2 0; type revolute -> fixed
- joint Left_Shoulder_Roll: origin xyz=0 0.047 0 rpy=0.0 0 0 -> xyz=0 0.047 0 rpy=-1.35 0 0; type revolute -> fixed
- joint Right_Elbow_Pitch: type revolute -> fixed
- joint Right_Elbow_Yaw: origin xyz=0 -0.1471 0 rpy=0 0 0 -> xyz=0 -0.1471 0 rpy=0 0 0.5; type revolute -> fixed
- joint Right_Shoulder_Pitch: origin xyz=0.0575 -0.1063 0.219 rpy=0 0 0 -> xyz=0.0575 -0.1063 0.219 rpy=0 0.2 0; type revolute -> fixed
- joint Right_Shoulder_Roll: origin xyz=0 -0.047 0 rpy=0 0 0 -> xyz=0 -0.047 0 rpy=1.35 0 0; type revolute -> fixed

File: IsaacGymRL/resources/T1/T1_collision_mesh.urdf (robot description, URDF)
Before this commit: robot T1, 24 links, 23 joints
Links:
- link H2: geometry collision mesh filename=meshes/H2.STL; visual mesh filename=meshes/H2.STL
Joints:
- joint Left_Elbow_Yaw: origin xyz=0 0.1471 0 rpy=0 0 0 -> xyz=0 0.1471 0 rpy=0 0 -0.5
- joint Left_Shoulder_Pitch: origin xyz=0.0575 0.1063 0.219 rpy=0 0 0 -> xyz=0.0575 0.1063 0.219 rpy=0 0.2 0
- joint Left_Shoulder_Roll: origin xyz=0 0.047 0 rpy=0.0 0 0 -> xyz=0 0.047 0 rpy=-1.35 0 0
- joint Right_Elbow_Yaw: origin xyz=0 -0.1471 0 rpy=0 0 0 -> xyz=0 -0.1471 0 rpy=0 0 0.5
- joint Right_Shoulder_Pitch: origin xyz=0.0575 -0.1063 0.219 rpy=0 0 0 -> xyz=0.0575 -0.1063 0.219 rpy=0 0.2 0
- joint Right_Shoulder_Roll: origin xyz=0 -0.047 0 rpy=0 0 0 -> xyz=0 -0.047 0 rpy=1.35 0 0

File: IsaacGymRL/resources/T1/T1_locomotion.urdf (robot description, URDF)
Before this commit: robot T1, 24 links, 23 joints
Links:
- link AL1: geometry visual mesh filename=meshes/AL1.STL
- link AL2: geometry visual mesh filename=meshes/AL2.STL
- link AL3: geometry visual mesh filename=meshes/AL3.STL
- link AR1: geometry visual mesh filename=meshes/AR1.STL
- link AR2: geometry visual mesh filename=meshes/AR2.STL
- link AR3: geometry visual mesh filename=meshes/AR3.STL
- link Ankle_Cross_Left: geometry visual mesh filename=meshes/Ankle_Cross_Left.STL
- link Ankle_Cross_Right: geometry visual mesh filename=meshes/Ankle_Cross_Right.STL
- link H1: geometry visual mesh filename=meshes/H1.STL
- link H2: geometry visual mesh filename=meshes/H2.STL
- link Hip_Pitch_Left: geometry visual mesh filename=meshes/Hip_Pitch_Left.STL
- link Hip_Pitch_Right: geometry visual mesh filename=meshes/Hip_Pitch_Right.STL
- link Hip_Roll_Left: geometry visual mesh filename=meshes/Hip_Roll_Left.STL
- link Hip_Roll_Right: geometry visual mesh filename=meshes/Hip_Roll_Right.STL
- link Hip_Yaw_Left: geometry collision cylinder length=0.12 radius=0.05; visual mesh filename=meshes/Hip_Yaw_Left.STL
- link Hip_Yaw_Right: geometry collision cylinder length=0.12 radius=0.05; visual mesh filename=meshes/Hip_Yaw_Right.STL
- link Shank_Left: geometry collision mesh filename=meshes/Shank_Left.STL scale=1 1 0.8; visual mesh filename=meshes/Shank_Left.STL
- link Shank_Right: geometry collision mesh filename=meshes/Shank_Right.STL scale=1 1 0.8; visual mesh filename=meshes/Shank_Right.STL
- link Trunk: geometry collision box size=0.15 0.2 0.3; visual mesh filename=meshes/Trunk.STL
- link Waist: geometry visual mesh filename=meshes/Waist.STL
- link left_hand_link: geometry visual mesh filename=meshes/left_hand_link.STL
- link right_hand_link: geometry visual mesh filename=meshes/right_hand_link.STL
Joints:
- joint AAHead_yaw: type revolute -> fixed
- joint Head_pitch: type revolute -> fixed
- joint Left_Elbow_Pitch: type revolute -> fixed
- joint Left_Elbow_Yaw: origin xyz=0 0.1471 0 rpy=0 0 0 -> xyz=0 0.1471 0 rpy=0 0 -0.5; type revolute -> fixed
- joint Left_Shoulder_Pitch: origin xyz=0.0575 0.1063 0.219 rpy=0 0 0 -> xyz=0.0575 0.1063 0.219 rpy=0 0.2 0; type revolute -> fixed
- joint Left_Shoulder_Roll: origin xyz=0 0.047 0 rpy=0.0 0 0 -> xyz=0 0.047 0 rpy=-1.35 0 0; type revolute -> fixed
- joint Right_Elbow_Pitch: type revolute -> fixed
- joint Right_Elbow_Yaw: origin xyz=0 -0.1471 0 rpy=0 0 0 -> xyz=0 -0.1471 0 rpy=0 0 0.5; type revolute -> fixed
- joint Right_Shoulder_Pitch: origin xyz=0.0575 -0.1063 0.219 rpy=0 0 0 -> xyz=0.0575 -0.1063 0.219 rpy=0 0.2 0; type revolute -> fixed
- joint Right_Shoulder_Roll: origin xyz=0 -0.047 0 rpy=0 0 0 -> xyz=0 -0.047 0 rpy=1.35 0 0; type revolute -> fixed

File: IsaacGymRL/resources/T1/T1_locomotion_all_joints_simple.urdf (robot description, URDF)
Before this commit: robot T1, 24 links, 23 joints
Joints:
- joint Left_Knee_Pitch: limit lower=-0.199 upper=2.34 effort=60 velocity=14.7 -> lower=0.0 upper=2.34 effort=60 velocity=14.7
- joint Right_Knee_Pitch: limit lower=-0.199 upper=2.34 effort=60 velocity=14.7 -> lower=0.0 upper=2.34 effort=60 velocity=14.7

File: IsaacGymRL/resources/T1/T1_locomotion_feet_box.urdf (robot description, URDF)
Before this commit: robot T1, 24 links, 23 joints
Links:
- link AL1: geometry visual mesh filename=meshes/AL1.STL
- link AL2: geometry visual mesh filename=meshes/AL2.STL
- link AL3: geometry visual mesh filename=meshes/AL3.STL
- link AR1: geometry visual mesh filename=meshes/AR1.STL
- link AR2: geometry visual mesh filename=meshes/AR2.STL
- link AR3: geometry visual mesh filename=meshes/AR3.STL
- link Ankle_Cross_Left: geometry visual mesh filename=meshes/Ankle_Cross_Left.STL
- link Ankle_Cross_Right: geometry visual mesh filename=meshes/Ankle_Cross_Right.STL
- link H1: geometry visual mesh filename=meshes/H1.STL
- link H2: geometry visual mesh filename=meshes/H2.STL
- link Hip_Pitch_Left: geometry visual mesh filename=meshes/Hip_Pitch_Left.STL
- link Hip_Pitch_Right: geometry visual mesh filename=meshes/Hip_Pitch_Right.STL
- link Hip_Roll_Left: geometry visual mesh filename=meshes/Hip_Roll_Left.STL
- link Hip_Roll_Right: geometry visual mesh filename=meshes/Hip_Roll_Right.STL
- link Hip_Yaw_Left: geometry collision cylinder length=0.16 radius=0.05; visual mesh filename=meshes/Hip_Yaw_Left.STL
- link Hip_Yaw_Right: geometry collision cylinder length=0.16 radius=0.05; visual mesh filename=meshes/Hip_Yaw_Right.STL
- link Shank_Left: geometry collision box size=0.01 0.10 0.05; collision box size=0.1 0.14 0.12
- link Shank_Right: geometry collision box size=0.01 0.10 0.05; collision box size=0.1 0.14 0.12
- link Trunk: geometry collision box size=0.15 0.2 0.3; visual mesh filename=meshes/Trunk.STL
- link Waist: geometry visual mesh filename=meshes/Waist.STL
- link left_foot_link: geometry collision box size=0.223 0.1 0.03; visual mesh filename=meshes/left_foot_link.STL
- link left_hand_link: geometry visual mesh filename=meshes/left_hand_link.STL
- link right_foot_link: geometry collision box size=0.223 0.1 0.03; visual mesh filename=meshes/right_foot_link.STL
- link right_hand_link: geometry visual mesh filename=meshes/right_hand_link.STL
Joints:
- joint AAHead_yaw: type revolute -> fixed
- joint Head_pitch: type revolute -> fixed
- joint Left_Elbow_Pitch: type revolute -> fixed
- joint Left_Elbow_Yaw: origin xyz=0 0.1471 0 rpy=0 0 0 -> xyz=0 0.1471 0 rpy=0 0 -0.5; type revolute -> fixed
- joint Left_Shoulder_Pitch: origin xyz=0.0575 0.1063 0.219 rpy=0 0 0 -> xyz=0.0575 0.1063 0.219 rpy=0 0.2 0; type revolute -> fixed
- joint Left_Shoulder_Roll: origin xyz=0 0.047 0 rpy=0.0 0 0 -> xyz=0 0.047 0 rpy=-1.35 0 0; type revolute -> fixed
- joint Right_Elbow_Pitch: type revolute -> fixed
- joint Right_Elbow_Yaw: origin xyz=0 -0.1471 0 rpy=0 0 0 -> xyz=0 -0.1471 0 rpy=0 0 0.5; type revolute -> fixed
- joint Right_Shoulder_Pitch: origin xyz=0.0575 -0.1063 0.219 rpy=0 0 0 -> xyz=0.0575 -0.1063 0.219 rpy=0 0.2 0; type revolute -> fixed
- joint Right_Shoulder_Roll: origin xyz=0 -0.047 0 rpy=0 0 0 -> xyz=0 -0.047 0 rpy=1.35 0 0; type revolute -> fixed
