Commit message: Update K1 and T1 position limits
- Those are based on the measured limits of the real robots

File: IsaacGymRL/resources/K1/Ball_K1_locomotion_feet_box_left_bias.urdf (robot description, URDF)
Before this commit: robot K1, 23 links, 22 joints
Joints:
- joint AAHead_yaw: limit lower=-1. upper=1. effort=6 velocity=18 -> lower=-1.04 upper=1.04 effort=6 velocity=18
- joint ALeft_Shoulder_Pitch: limit lower=-3.316 upper=1.22 effort=14 velocity=18 -> lower=-2.95 upper=1.22 effort=14 velocity=18
- joint ARight_Shoulder_Pitch: limit lower=-3.316 upper=1.22 effort=14 velocity=18 -> lower=-2.95 upper=1.22 effort=14 velocity=18
- joint Head_pitch: limit lower=-0.349 upper=0.855 effort=6 velocity=18 -> lower=-0.3 upper=0.89 effort=6 velocity=18
- joint Left_Elbow_Pitch: limit lower=-2.27 upper=2.27 effort=14 velocity=18 -> lower=-1.9 upper=1.9 effort=14 velocity=18
- joint Left_Elbow_Yaw: limit lower=-2.44 upper=0 effort=14 velocity=18 -> lower=-2.25 upper=0.78 effort=14 velocity=18
- joint Left_Hip_Roll: limit lower=-0.4 upper=1.57 effort=35 velocity=12.9 -> lower=-0.38 upper=1.57 effort=35 velocity=12.9
- joint Left_Hip_Yaw: limit lower=-1. upper=1. effort=20 velocity=18.1 -> lower=-1.03 upper=1.03 effort=20 velocity=18.1
- joint Left_Knee_Pitch: limit lower=0. upper=2.23 effort=40 velocity=12.5 -> lower=0. upper=2.35 effort=40 velocity=12.5
- joint Right_Elbow_Pitch: limit lower=-2.27 upper=2.27 effort=14 velocity=18 -> lower=-1.9 upper=1.9 effort=14 velocity=18
- joint Right_Elbow_Yaw: limit lower=0 upper=2.44 effort=14 velocity=18 -> lower=-0.78 upper=2.25 effort=14 velocity=18
- joint Right_Hip_Roll: limit lower=-1.57 upper=0.4 effort=35 velocity=12.9 -> lower=-1.57 upper=0.38 effort=35 velocity=12.9
- joint Right_Hip_Yaw: limit lower=-1. upper=1. effort=20 velocity=18.1 -> lower=-1.03 upper=1.03 effort=20 velocity=18.1
- joint Right_Knee_Pitch: limit lower=0. upper=2.23 effort=40 velocity=12.5 -> lower=0. upper=2.35 effort=40 velocity=12.5

File: IsaacGymRL/resources/K1/Ball_K1_locomotion_feet_box_right_bias.urdf (robot description, URDF)
Before this commit: robot K1, 23 links, 22 joints
Joints:
- joint AAHead_yaw: limit lower=-1. upper=1. effort=6 velocity=18 -> lower=-1.04 upper=1.04 effort=6 velocity=18
- joint ALeft_Shoulder_Pitch: limit lower=-3.316 upper=1.22 effort=14 velocity=18 -> lower=-2.95 upper=1.22 effort=14 velocity=18
- joint ARight_Shoulder_Pitch: limit lower=-3.316 upper=1.22 effort=14 velocity=18 -> lower=-2.95 upper=1.22 effort=14 velocity=18
- joint Head_pitch: limit lower=-0.349 upper=0.855 effort=6 velocity=18 -> lower=-0.3 upper=0.89 effort=6 velocity=18
- joint Left_Elbow_Pitch: limit lower=-2.27 upper=2.27 effort=14 velocity=18 -> lower=-1.9 upper=1.9 effort=14 velocity=18
- joint Left_Elbow_Yaw: limit lower=-2.44 upper=0 effort=14 velocity=18 -> lower=-2.25 upper=0.78 effort=14 velocity=18
- joint Left_Hip_Roll: limit lower=-0.4 upper=1.57 effort=35 velocity=12.9 -> lower=-0.38 upper=1.57 effort=35 velocity=12.9
- joint Left_Hip_Yaw: limit lower=-1. upper=1. effort=20 velocity=18.1 -> lower=-1.03 upper=1.03 effort=20 velocity=18.1
- joint Left_Knee_Pitch: limit lower=0. upper=2.23 effort=40 velocity=12.5 -> lower=0. upper=2.35 effort=40 velocity=12.5
- joint Right_Elbow_Pitch: limit lower=-2.27 upper=2.27 effort=14 velocity=18 -> lower=-1.9 upper=1.9 effort=14 velocity=18
- joint Right_Elbow_Yaw: limit lower=0 upper=2.44 effort=14 velocity=18 -> lower=-0.78 upper=2.25 effort=14 velocity=18
- joint Right_Hip_Roll: limit lower=-1.57 upper=0.4 effort=35 velocity=12.9 -> lower=-1.57 upper=0.38 effort=35 velocity=12.9
- joint Right_Hip_Yaw: limit lower=-1. upper=1. effort=20 velocity=18.1 -> lower=-1.03 upper=1.03 effort=20 velocity=18.1
- joint Right_Knee_Pitch: limit lower=0. upper=2.23 effort=40 velocity=12.5 -> lower=0. upper=2.35 effort=40 velocity=12.5

File: IsaacGymRL/resources/K1/K1_arms_locomotion.urdf (robot description, URDF)
Before this commit: robot K1, 23 links, 22 joints
Joints:
- joint AAHead_yaw: limit lower=-1. upper=1. effort=6 velocity=18 -> lower=-1.04 upper=1.04 effort=6 velocity=18
- joint ALeft_Shoulder_Pitch: limit lower=-3.316 upper=1.22 effort=14 velocity=18 -> lower=-2.95 upper=1.22 effort=14 velocity=18
- joint ARight_Shoulder_Pitch: limit lower=-3.316 upper=1.22 effort=14 velocity=18 -> lower=-2.95 upper=1.22 effort=14 velocity=18
- joint Head_pitch: limit lower=-0.349 upper=0.855 effort=6 velocity=18 -> lower=-0.3 upper=0.89 effort=6 velocity=18
- joint Left_Elbow_Pitch: limit lower=-2.27 upper=2.27 effort=14 velocity=18 -> lower=-1.9 upper=1.9 effort=14 velocity=18
- joint Left_Elbow_Yaw: limit lower=-2.44 upper=0 effort=14 velocity=18 -> lower=-2.25 upper=0.78 effort=14 velocity=18
- joint Left_Hip_Roll: limit lower=-0.4 upper=1.57 effort=35 velocity=12.9 -> lower=-0.38 upper=1.57 effort=35 velocity=12.9
- joint Left_Hip_Yaw: limit lower=-1. upper=1. effort=20 velocity=18.1 -> lower=-1.03 upper=1.03 effort=20 velocity=18.1
- joint Left_Knee_Pitch: limit lower=0. upper=2.23 effort=40 velocity=12.5 -> lower=0. upper=2.35 effort=40 velocity=12.5
- joint Right_Elbow_Pitch: limit lower=-2.27 upper=2.27 effort=14 velocity=18 -> lower=-1.9 upper=1.9 effort=14 velocity=18
- joint Right_Elbow_Yaw: limit lower=0 upper=2.44 effort=14 velocity=18 -> lower=-0.78 upper=2.25 effort=14 velocity=18
- joint Right_Hip_Roll: limit lower=-1.57 upper=0.4 effort=35 velocity=12.9 -> lower=-1.57 upper=0.38 effort=35 velocity=12.9
- joint Right_Hip_Yaw: limit lower=-1. upper=1. effort=20 velocity=18.1 -> lower=-1.03 upper=1.03 effort=20 velocity=18.1
- joint Right_Knee_Pitch: limit lower=0. upper=2.23 effort=40 velocity=12.5 -> lower=0. upper=2.35 effort=40 velocity=12.5

File: IsaacGymRL/resources/K1/K1_arms_locomotion_feet_box.urdf (robot description, URDF)
Before this commit: robot K1, 23 links, 22 joints
Joints:
- joint AAHead_yaw: limit lower=-1. upper=1. effort=6 velocity=18 -> lower=-1.04 upper=1.04 effort=6 velocity=18
- joint ALeft_Shoulder_Pitch: limit lower=-3.316 upper=1.22 effort=14 velocity=18 -> lower=-2.95 upper=1.22 effort=14 velocity=18
- joint ARight_Shoulder_Pitch: limit lower=-3.316 upper=1.22 effort=14 velocity=18 -> lower=-2.95 upper=1.22 effort=14 velocity=18
- joint Head_pitch: limit lower=-0.349 upper=0.855 effort=6 velocity=18 -> lower=-0.3 upper=0.89 effort=6 velocity=18
- joint Left_Elbow_Pitch: limit lower=-2.27 upper=2.27 effort=14 velocity=18 -> lower=-1.9 upper=1.9 effort=14 velocity=18
- joint Left_Elbow_Yaw: limit lower=-2.44 upper=0 effort=14 velocity=18 -> lower=-2.25 upper=0.78 effort=14 velocity=18
- joint Left_Hip_Roll: limit lower=-0.4 upper=1.57 effort=35 velocity=12.9 -> lower=-0.38 upper=1.57 effort=35 velocity=12.9
- joint Left_Hip_Yaw: limit lower=-1. upper=1. effort=20 velocity=18.1 -> lower=-1.03 upper=1.03 effort=20 velocity=18.1
- joint Left_Knee_Pitch: limit lower=0. upper=2.23 effort=40 velocity=12.5 -> lower=0. upper=2.35 effort=40 velocity=12.5
- joint Right_Elbow_Pitch: limit lower=-2.27 upper=2.27 effort=14 velocity=18 -> lower=-1.9 upper=1.9 effort=14 velocity=18
- joint Right_Elbow_Yaw: limit lower=0 upper=2.44 effort=14 velocity=18 -> lower=-0.78 upper=2.25 effort=14 velocity=18
- joint Right_Hip_Roll: limit lower=-1.57 upper=0.4 effort=35 velocity=12.9 -> lower=-1.57 upper=0.38 effort=35 velocity=12.9
- joint Right_Hip_Yaw: limit lower=-1. upper=1. effort=20 velocity=18.1 -> lower=-1.03 upper=1.03 effort=20 velocity=18.1
- joint Right_Knee_Pitch: limit lower=0. upper=2.23 effort=40 velocity=12.5 -> lower=0. upper=2.35 effort=40 velocity=12.5

File: IsaacGymRL/resources/K1/K1_locomotion.urdf (robot description, URDF)
Before this commit: robot K1, 23 links, 22 joints
Joints:
- joint AAHead_yaw: limit lower=-1. upper=1. effort=6 velocity=18 -> lower=-1.04 upper=1.04 effort=6 velocity=18
- joint ALeft_Shoulder_Pitch: limit lower=-3.316 upper=1.22 effort=14 velocity=18 -> lower=-2.95 upper=1.22 effort=14 velocity=18
- joint ARight_Shoulder_Pitch: limit lower=-3.316 upper=1.22 effort=14 velocity=18 -> lower=-2.95 upper=1.22 effort=14 velocity=18
- joint Head_pitch: limit lower=-0.349 upper=0.855 effort=6 velocity=18 -> lower=-0.3 upper=0.89 effort=6 velocity=18
- joint Left_Elbow_Pitch: limit lower=-2.27 upper=2.27 effort=14 velocity=18 -> lower=-1.9 upper=1.9 effort=14 velocity=18
- joint Left_Elbow_Yaw: limit lower=-2.44 upper=0 effort=14 velocity=18 -> lower=-2.25 upper=0.78 effort=14 velocity=18
- joint Left_Hip_Roll: limit lower=-0.4 upper=1.57 effort=35 velocity=12.9 -> lower=-0.38 upper=1.57 effort=35 velocity=12.9
- joint Left_Hip_Yaw: limit lower=-1. upper=1. effort=20 velocity=18.1 -> lower=-1.03 upper=1.03 effort=20 velocity=18.1
- joint Left_Knee_Pitch: limit lower=0. upper=2.23 effort=40 velocity=12.5 -> lower=0. upper=2.35 effort=40 velocity=12.5
- joint Right_Elbow_Pitch: limit lower=-2.27 upper=2.27 effort=14 velocity=18 -> lower=-1.9 upper=1.9 effort=14 velocity=18
- joint Right_Elbow_Yaw: limit lower=0 upper=2.44 effort=14 velocity=18 -> lower=-0.78 upper=2.25 effort=14 velocity=18
- joint Right_Hip_Roll: limit lower=-1.57 upper=0.4 effort=35 velocity=12.9 -> lower=-1.57 upper=0.38 effort=35 velocity=12.9
- joint Right_Hip_Yaw: limit lower=-1. upper=1. effort=20 velocity=18.1 -> lower=-1.03 upper=1.03 effort=20 velocity=18.1
- joint Right_Knee_Pitch: limit lower=0. upper=2.23 effort=40 velocity=12.5 -> lower=0. upper=2.35 effort=40 velocity=12.5

File: IsaacGymRL/resources/K1/K1_locomotion_all_joints_mesh.urdf (robot description, URDF)
Before this commit: robot K1, 23 links, 22 joints
Joints:
- joint AAHead_yaw: limit lower=-1. upper=1. effort=6 velocity=18 -> lower=-1.04 upper=1.04 effort=6 velocity=18
- joint ALeft_Shoulder_Pitch: limit lower=-3.316 upper=1.22 effort=14 velocity=18 -> lower=-2.95 upper=1.22 effort=14 velocity=18
- joint ARight_Shoulder_Pitch: limit lower=-3.316 upper=1.22 effort=14 velocity=18 -> lower=-2.95 upper=1.22 effort=14 velocity=18
- joint Head_pitch: limit lower=-0.349 upper=0.855 effort=6 velocity=18 -> lower=-0.3 upper=0.89 effort=6 velocity=18
- joint Left_Elbow_Pitch: limit lower=-2.27 upper=2.27 effort=14 velocity=18 -> lower=-1.9 upper=1.9 effort=14 velocity=18
- joint Left_Elbow_Yaw: limit lower=-2.44 upper=0 effort=14 velocity=18 -> lower=-2.25 upper=0.78 effort=14 velocity=18
- joint Left_Hip_Roll: limit lower=-0.4 upper=1.57 effort=35 velocity=12.9 -> lower=-0.38 upper=1.57 effort=35 velocity=12.9
- joint Left_Hip_Yaw: limit lower=-1. upper=1. effort=20 velocity=18.1 -> lower=-1.03 upper=1.03 effort=20 velocity=18.1
- joint Left_Knee_Pitch: limit lower=0. upper=2.23 effort=40 velocity=12.5 -> lower=0. upper=2.35 effort=40 velocity=12.5
- joint Right_Elbow_Pitch: limit lower=-2.27 upper=2.27 effort=14 velocity=18 -> lower=-1.9 upper=1.9 effort=14 velocity=18
- joint Right_Elbow_Yaw: limit lower=0 upper=2.44 effort=14 velocity=18 -> lower=-0.78 upper=2.25 effort=14 velocity=18
- joint Right_Hip_Roll: limit lower=-1.57 upper=0.4 effort=35 velocity=12.9 -> lower=-1.57 upper=0.38 effort=35 velocity=12.9
- joint Right_Hip_Yaw: limit lower=-1. upper=1. effort=20 velocity=18.1 -> lower=-1.03 upper=1.03 effort=20 velocity=18.1
- joint Right_Knee_Pitch: limit lower=0. upper=2.23 effort=40 velocity=12.5 -> lower=0. upper=2.35 effort=40 velocity=12.5

File: IsaacGymRL/resources/K1/K1_locomotion_all_joints_simple.urdf (robot description, URDF)
Before this commit: robot K1, 23 links, 22 joints
Joints:
- joint AAHead_yaw: limit lower=-1. upper=1. effort=6 velocity=18 -> lower=-1.04 upper=1.04 effort=6 velocity=18
- joint ALeft_Shoulder_Pitch: limit lower=-3.316 upper=1.22 effort=14 velocity=18 -> lower=-2.95 upper=1.22 effort=14 velocity=18
- joint ARight_Shoulder_Pitch: limit lower=-3.316 upper=1.22 effort=14 velocity=18 -> lower=-2.95 upper=1.22 effort=14 velocity=18
- joint Head_pitch: limit lower=-0.349 upper=0.855 effort=6 velocity=18 -> lower=-0.3 upper=0.89 effort=6 velocity=18
- joint Left_Elbow_Pitch: limit lower=-2.27 upper=2.27 effort=14 velocity=18 -> lower=-1.9 upper=1.9 effort=14 velocity=18
- joint Left_Elbow_Yaw: limit lower=-2.44 upper=0 effort=14 velocity=18 -> lower=-2.25 upper=0.78 effort=14 velocity=18
- joint Left_Hip_Roll: limit lower=-0.4 upper=1.57 effort=35 velocity=12.9 -> lower=-0.38 upper=1.57 effort=35 velocity=12.9
- joint Left_Hip_Yaw: limit lower=-1. upper=1. effort=20 velocity=18.1 -> lower=-1.03 upper=1.03 effort=20 velocity=18.1
- joint Left_Knee_Pitch: limit lower=0. upper=2.23 effort=40 velocity=12.5 -> lower=0. upper=2.35 effort=40 velocity=12.5
- joint Right_Elbow_Pitch: limit lower=-2.27 upper=2.27 effort=14 velocity=18 -> lower=-1.9 upper=1.9 effort=14 velocity=18
- joint Right_Elbow_Yaw: limit lower=0 upper=2.44 effort=14 velocity=18 -> lower=-0.78 upper=2.25 effort=14 velocity=18
- joint Right_Hip_Roll: limit lower=-1.57 upper=0.4 effort=35 velocity=12.9 -> lower=-1.57 upper=0.38 effort=35 velocity=12.9
- joint Right_Hip_Yaw: limit lower=-1. upper=1. effort=20 velocity=18.1 -> lower=-1.03 upper=1.03 effort=20 velocity=18.1
- joint Right_Knee_Pitch: limit lower=0. upper=2.23 effort=40 velocity=12.5 -> lower=0. upper=2.35 effort=40 velocity=12.5

File: IsaacGymRL/resources/K1/K1_locomotion_all_joints_simple_2.urdf (robot description, URDF)
Before this commit: robot K1, 23 links, 22 joints
Joints:
- joint AAHead_yaw: limit lower=-1. upper=1. effort=6 velocity=18 -> lower=-1.04 upper=1.04 effort=6 velocity=18
- joint ALeft_Shoulder_Pitch: limit lower=-3.316 upper=1.22 effort=14 velocity=18 -> lower=-2.95 upper=1.22 effort=14 velocity=18
- joint ARight_Shoulder_Pitch: limit lower=-3.316 upper=1.22 effort=14 velocity=18 -> lower=-2.95 upper=1.22 effort=14 velocity=18
- joint Head_pitch: limit lower=-0.349 upper=0.855 effort=6 velocity=18 -> lower=-0.3 upper=0.89 effort=6 velocity=18
- joint Left_Elbow_Pitch: limit lower=-2.27 upper=2.27 effort=14 velocity=18 -> lower=-1.9 upper=1.9 effort=14 velocity=18
- joint Left_Elbow_Yaw: limit lower=-2.44 upper=0 effort=14 velocity=18 -> lower=-2.25 upper=0.78 effort=14 velocity=18
- joint Left_Hip_Roll: limit lower=-0.4 upper=1.57 effort=35 velocity=12.9 -> lower=-0.38 upper=1.57 effort=35 velocity=12.9
- joint Left_Hip_Yaw: limit lower=-1. upper=1. effort=20 velocity=18.1 -> lower=-1.03 upper=1.03 effort=20 velocity=18.1
- joint Left_Knee_Pitch: limit lower=0. upper=2.23 effort=40 velocity=12.5 -> lower=0. upper=2.35 effort=40 velocity=12.5
- joint Right_Elbow_Pitch: limit lower=-2.27 upper=2.27 effort=14 velocity=18 -> lower=-1.9 upper=1.9 effort=14 velocity=18
- joint Right_Elbow_Yaw: limit lower=0 upper=2.44 effort=14 velocity=18 -> lower=-0.78 upper=2.25 effort=14 velocity=18
- joint Right_Hip_Roll: limit lower=-1.57 upper=0.4 effort=35 velocity=12.9 -> lower=-1.57 upper=0.38 effort=35 velocity=12.9
- joint Right_Hip_Yaw: limit lower=-1. upper=1. effort=20 velocity=18.1 -> lower=-1.03 upper=1.03 effort=20 velocity=18.1
- joint Right_Knee_Pitch: limit lower=0. upper=2.23 effort=40 velocity=12.5 -> lower=0. upper=2.35 effort=40 velocity=12.5

File: IsaacGymRL/resources/K1/K1_locomotion_feet_box.urdf (robot description, URDF)
Before this commit: robot K1, 23 links, 22 joints
Joints:
- joint AAHead_yaw: limit lower=-1. upper=1. effort=6 velocity=18 -> lower=-1.04 upper=1.04 effort=6 velocity=18
- joint ALeft_Shoulder_Pitch: limit lower=-3.316 upper=1.22 effort=14 velocity=18 -> lower=-2.95 upper=1.22 effort=14 velocity=18
- joint ARight_Shoulder_Pitch: limit lower=-3.316 upper=1.22 effort=14 velocity=18 -> lower=-2.95 upper=1.22 effort=14 velocity=18
- joint Head_pitch: limit lower=-0.349 upper=0.855 effort=6 velocity=18 -> lower=-0.3 upper=0.89 effort=6 velocity=18
- joint Left_Elbow_Pitch: limit lower=-2.27 upper=2.27 effort=14 velocity=18 -> lower=-1.9 upper=1.9 effort=14 velocity=18
- joint Left_Elbow_Yaw: limit lower=-2.44 upper=0 effort=14 velocity=18 -> lower=-2.25 upper=0.78 effort=14 velocity=18
- joint Left_Hip_Roll: limit lower=-0.4 upper=1.57 effort=35 velocity=12.9 -> lower=-0.38 upper=1.57 effort=35 velocity=12.9
- joint Left_Hip_Yaw: limit lower=-1. upper=1. effort=20 velocity=18.1 -> lower=-1.03 upper=1.03 effort=20 velocity=18.1
- joint Left_Knee_Pitch: limit lower=0. upper=2.23 effort=40 velocity=12.5 -> lower=0. upper=2.35 effort=40 velocity=12.5
- joint Right_Elbow_Pitch: limit lower=-2.27 upper=2.27 effort=14 velocity=18 -> lower=-1.9 upper=1.9 effort=14 velocity=18
- joint Right_Elbow_Yaw: limit lower=0 upper=2.44 effort=14 velocity=18 -> lower=-0.78 upper=2.25 effort=14 velocity=18
- joint Right_Hip_Roll: limit lower=-1.57 upper=0.4 effort=35 velocity=12.9 -> lower=-1.57 upper=0.38 effort=35 velocity=12.9
- joint Right_Hip_Yaw: limit lower=-1. upper=1. effort=20 velocity=18.1 -> lower=-1.03 upper=1.03 effort=20 velocity=18.1
- joint Right_Knee_Pitch: limit lower=0. upper=2.23 effort=40 velocity=12.5 -> lower=0. upper=2.35 effort=40 velocity=12.5

File: IsaacGymRL/resources/T1/Ball_T1_locomotion_feet_box_left_bias.urdf (robot description, URDF)
Before this commit: robot T1, 24 links, 23 joints
Joints:
- joint Head_pitch: limit lower=-0.3491 upper=0.8552 effort=7 velocity=12.56 -> lower=-0.38 upper=1.04 effort=7 velocity=12.56
- joint Left_Elbow_Yaw: limit lower=-2.1402 upper=1.6844 effort=18 velocity=18 -> lower=-2.09 upper=1.66 effort=18 velocity=18
- joint Left_Hip_Pitch: limit lower=-3.0020 upper=2.2166 effort=45 velocity=15.2 -> lower=-3.0020 upper=2.23 effort=45 velocity=15.2
- joint Left_Hip_Roll: limit lower=-0.55 upper=1.57 effort=25 velocity=7.1 -> lower=-0.4 upper=1.57 effort=25 velocity=7.1
- joint Left_Hip_Yaw: limit lower=-1 upper=1 effort=25 velocity=7.1 -> lower=-1.08 upper=1.08 effort=25 velocity=7.1
- joint Left_Knee_Pitch: limit lower=0.0 upper=2.34 effort=60 velocity=14.7 -> lower=0.0 upper=2.18 effort=60 velocity=14.7
- joint Left_Shoulder_Pitch: limit lower=-3.29 upper=1.18 effort=18 velocity=18 -> lower=-3.31 upper=1.22 effort=18 velocity=18
- joint Right_Elbow_Yaw: limit lower=-1.6844 upper=2.1402 effort=18 velocity=18 -> lower=-1.66 upper=2.06 effort=18 velocity=18
- joint Right_Hip_Pitch: limit lower=-3.0020 upper=2.2166 effort=45 velocity=15.2 -> lower=-3.0020 upper=2.23 effort=45 velocity=15.2
- joint Right_Hip_Roll: limit lower=-1.57 upper=0.55 effort=25 velocity=7.1 -> lower=-1.57 upper=0.4 effort=25 velocity=7.1
- joint Right_Hip_Yaw: limit lower=-1 upper=1 effort=25 velocity=7.1 -> lower=-1.08 upper=1.08 effort=25 velocity=7.1
- joint Right_Knee_Pitch: limit lower=0.0 upper=2.34 effort=60 velocity=14.7 -> lower=0.0 upper=2.18 effort=60 velocity=14.7
- joint Right_Shoulder_Pitch: limit lower=-3.29 upper=1.1868 effort=18 velocity=18 -> lower=-3.31 upper=1.22 effort=18 velocity=18
- joint Waist: limit lower=-1.57 upper=1.57 effort=25 velocity=7.1 -> lower=-1.04 upper=1.04 effort=25 velocity=7.1

File: IsaacGymRL/resources/T1/Ball_T1_locomotion_feet_box_right_bias.urdf (robot description, URDF)
Before this commit: robot T1, 24 links, 23 joints
Joints:
- joint Head_pitch: limit lower=-0.3491 upper=0.8552 effort=7 velocity=12.56 -> lower=-0.38 upper=1.04 effort=7 velocity=12.56
- joint Left_Elbow_Yaw: limit lower=-2.1402 upper=1.6844 effort=18 velocity=18 -> lower=-2.09 upper=1.66 effort=18 velocity=18
- joint Left_Hip_Pitch: limit lower=-3.0020 upper=2.2166 effort=45 velocity=15.2 -> lower=-3.0020 upper=2.23 effort=45 velocity=15.2
- joint Left_Hip_Roll: limit lower=-0.55 upper=1.57 effort=25 velocity=7.1 -> lower=-0.4 upper=1.57 effort=25 velocity=7.1
- joint Left_Hip_Yaw: limit lower=-1 upper=1 effort=25 velocity=7.1 -> lower=-1.08 upper=1.08 effort=25 velocity=7.1
- joint Left_Knee_Pitch: limit lower=0.0 upper=2.34 effort=60 velocity=14.7 -> lower=0.0 upper=2.18 effort=60 velocity=14.7
- joint Left_Shoulder_Pitch: limit lower=-3.29 upper=1.18 effort=18 velocity=18 -> lower=-3.31 upper=1.22 effort=18 velocity=18
- joint Right_Elbow_Yaw: limit lower=-1.6844 upper=2.1402 effort=18 velocity=18 -> lower=-1.66 upper=2.09 effort=18 velocity=18
- joint Right_Hip_Pitch: limit lower=-3.0020 upper=2.2166 effort=45 velocity=15.2 -> lower=-3.0020 upper=2.23 effort=45 velocity=15.2
- joint Right_Hip_Roll: limit lower=-1.57 upper=0.55 effort=25 velocity=7.1 -> lower=-1.57 upper=0.4 effort=25 velocity=7.1
- joint Right_Hip_Yaw: limit lower=-1 upper=1 effort=25 velocity=7.1 -> lower=-1.08 upper=1.08 effort=25 velocity=7.1
- joint Right_Knee_Pitch: limit lower=0.0 upper=2.34 effort=60 velocity=14.7 -> lower=0.0 upper=2.18 effort=60 velocity=14.7
- joint Right_Shoulder_Pitch: limit lower=-3.29 upper=1.1868 effort=18 velocity=18 -> lower=-3.31 upper=1.22 effort=18 velocity=18
- joint Waist: limit lower=-1.57 upper=1.57 effort=25 velocity=7.1 -> lower=-1.04 upper=1.04 effort=25 velocity=7.1

File: IsaacGymRL/resources/T1/T1_collision_mesh.urdf (robot description, URDF)
Before this commit: robot T1, 24 links, 23 joints
Joints:
- joint Head_pitch: limit lower=-0.3491 upper=0.8552 effort=7 velocity=12.56 -> lower=-0.38 upper=1.04 effort=7 velocity=12.56
- joint Left_Elbow_Yaw: limit lower=-2.1402 upper=1.6844 effort=18 velocity=18 -> lower=-2.09 upper=1.66 effort=18 velocity=18
- joint Left_Hip_Pitch: limit lower=-3.0020 upper=2.2166 effort=45 velocity=15.2 -> lower=-3.0020 upper=2.23 effort=45 velocity=15.2
- joint Left_Hip_Roll: limit lower=-0.55 upper=1.57 effort=25 velocity=7.1 -> lower=-0.4 upper=1.57 effort=25 velocity=7.1
- joint Left_Hip_Yaw: limit lower=-1 upper=1 effort=25 velocity=7.1 -> lower=-1.08 upper=1.08 effort=25 velocity=7.1
- joint Left_Knee_Pitch: limit lower=0.0 upper=2.34 effort=60 velocity=14.7 -> lower=0.0 upper=2.18 effort=60 velocity=14.7
- joint Left_Shoulder_Pitch: limit lower=-3.29 upper=1.18 effort=18 velocity=18 -> lower=-3.31 upper=1.22 effort=18 velocity=18
- joint Right_Elbow_Yaw: limit lower=-1.6844 upper=2.1402 effort=18 velocity=18 -> lower=-1.66 upper=2.09 effort=18 velocity=18
- joint Right_Hip_Pitch: limit lower=-3.0020 upper=2.2166 effort=45 velocity=15.2 -> lower=-3.0020 upper=2.23 effort=45 velocity=15.2
- joint Right_Hip_Roll: limit lower=-1.57 upper=0.55 effort=25 velocity=7.1 -> lower=-1.57 upper=0.4 effort=25 velocity=7.1
- joint Right_Hip_Yaw: limit lower=-1 upper=1 effort=25 velocity=7.1 -> lower=-1.08 upper=1.08 effort=25 velocity=7.1
- joint Right_Knee_Pitch: limit lower=0.0 upper=2.34 effort=60 velocity=14.7 -> lower=0.0 upper=2.18 effort=60 velocity=14.7
- joint Right_Shoulder_Pitch: limit lower=-3.29 upper=1.1868 effort=18 velocity=18 -> lower=-3.31 upper=1.22 effort=18 velocity=18
- joint Waist: limit lower=-1.57 upper=1.57 effort=25 velocity=7.1 -> lower=-1.04 upper=1.04 effort=25 velocity=7.1
